File: Design Files/ESC_rev0/ESC_rev0.kicad_pcb (KiCad board)
At the start: 4 copper layers, 100 x 75 mm, 175 parts, among them J1 Conn_01x08, J2 Conn_01x06, J3 Conn_01x03, J4 WP-BUTR, J5 WP-BUTR, J6 WP-BUTR, J7 Conn_01x04, J8 Conn_01x06, J9 USB_C_Receptacle_USB2.0_16P, Q1 HSBA15810C, Q2 HSBA15810C, Q3 HSBA15810C, Q4 HSBA15810C, Q5 HSBA15810C, Q6 HSBA15810C, SW1 Push Button, U1 XT60PW-M, U2 XH-2PWBPZ, U3 AMS1117-3.3, U4 STM32F405RGTx, U5 DRV8302DCA, U6 ESDCAN24-2BLY, U7 SN65HVD230, Y1 Crystal

Commit message: update 22
Board complete - not perfect for production, it is just a demo.  Generated gerber files through extensions, prepared some layout infos, updated the schematics with images. Note: due to a power outage, the last update had conflicts and the push was forced.
Parts:
- moved C28 45.5 mm to (83.8, 95.0)
- moved D1 45.5 mm to (110.5, 67.7)
- moved R26 45.5 mm to (113.3, 79.3)
- moved R29 45.5 mm to (113.3, 80.9)
- moved R31 45.5 mm to (120.5, 84.4)
- moved R5 45.5 mm to (83.4, 77.3)
- moved C17 45.5 mm to (58.4, 83.3)
- moved C2 45.5 mm to (107.0, 76.9)
- moved C3 45.5 mm to (47.9, 107.2)
- moved C48 45.5 mm to (49.1, 70.2)
- moved J7 45.5 mm to (40.0, 67.5)
- moved NT7 45.5 mm to (125.7, 112.1)
- moved R1 45.5 mm to (47.9, 108.7)
- moved R45 45.5 mm to (61.4, 107.4)
- moved R48 45.5 mm to (62.9, 107.4)
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Other:
- board text added: "0"
- board text added: "0 mm"
- board text added: "0,01 mm"
- board text added: "0,02"
- board text added: "0,03 mm"
- board text added: "0,07 mm"
- board text added: "0,1500 mm"
- board text added: "0,1600 mm / 0,1000 mm"
- board text added: "0,2 mm"
- board text added: "1"
- board text added: "1,03 mm"
- board text added: "1,6500 mm"
- board text added: "100,0000 mm x 75,0000 mm"
- board text added: "3,3"
- board text added: "4"
- board text added: "4,5"
- board text added: "B.Mask"
- board text added: "B.Paste"
- board text added: "B.Silkscreen"
- board text added: "BOARD CHARACTERISTICS"
- board text added: "Board Thickness:"
- board text added: "Board overall dimensions:"
- board text added: "Bottom Silk Screen"
- board text added: "Bottom Solder Mask"
- board text added: "Bottom Solder Paste"
- board text added: "Castellated pads:"
- board text added: "Color"
- board text added: "Copper Finish:"
- board text added: "Copper Layer Count:"
- board text added: "Dielectric"
- board text added: "Edge card connectors:"
- board text added: "Epsilon R"
- board text added: "F.Mask"
- board text added: "F.Paste"
- board text added: "F.Silkscreen"
- board text added: "FR4"
- board text added: "Green"
- board text added: "Impedance Control:"
- board text added: "L1_SGN_(Top).Cu"
- board text added: "L2_GND.Cu"
- board text added: "L3_GND.Cu"
- board text added: "L4_SGN_(Btm).Cu"
- board text added: "Layer Name"
- board text added: "Loss Tangent"
- board text added: "Material"
- board text added: "Min hole diameter:"
- board text added: "Min track/spacing:"
- board text added: "No"
- board text added: "None"
- board text added: "Not specified"
- board text added: "Plated Board Edge:"
- board text added: "Thickness (mm)"
- board text added: "Top Silk Screen"
- board text added: "Top Solder Mask"
- board text added: "Top Solder Paste"
- board text added: "Type"
- board text added: "copper"
- board text added: "core"
- board text added: "prepreg"
